File: 8052-IO.kicad_pcb (KiCad board)
At the start: 2 copper layers, 95 x 66 mm, 7 parts, among them J1 Conn_01x20_Pin, J2 Conn_01x20_Pin, J3 Conn_02x25_Odd_Even

Commit message: update
Parts:
- added J4: Conn_02x15_Odd_Even, Connector_PinHeader_2.54mm:PinHeader_2x15_P2.54mm_Horizontal, F.Cu at (117.3, 33.5)
- added J5: Conn_02x16_Odd_Even, Connector_PinHeader_2.54mm:PinHeader_2x15_P2.54mm_Horizontal, F.Cu at (158.0, 33.5)
- added U1: 82C55A, Package_DIP:DIP-40_W15.24mm, F.Cu at (116.0, 40.0)
- added U2: 74HC688, Package_SO:SOIC-20W_7.5x12.8mm_P1.27mm, F.Cu at (167.8, 82.4)
- added U3: 82C55A, Package_DIP:DIP-40_W15.24mm, F.Cu at (180.2, 39.9)
- moved H1 4.06 mm to (199.5, 30.5)
- moved H3 4.06 mm to (111.5, 30.5)
- moved J2 0.25 mm to (200.0, 39.9)
- moved H2 0.25 mm to (111.5, 93.5)
- moved H4 0.25 mm to (199.5, 93.5)
- moved J1 0.25 mm to (111.0, 40.0)
- moved J3 0.25 mm to (133.0, 95.0)
Connections:
- J1 pad 16: /~{WR} -> unconnected-(J1-Pin_16-Pad16)
- J1 pad 17: /~{RD} -> unconnected-(J1-Pin_17-Pad17)
- J2 pad 1: unconnected-(J2-Pin_1-Pad1) -> /CS0
- J2 pad 10: unconnected-(J2-Pin_10-Pad10) -> /CS9
- J2 pad 11: unconnected-(J2-Pin_11-Pad11) -> /CS10
- J2 pad 12: unconnected-(J2-Pin_12-Pad12) -> /CA11
- J2 pad 13: unconnected-(J2-Pin_13-Pad13) -> /CS12
- J2 pad 14: unconnected-(J2-Pin_14-Pad14) -> /CS13
- J2 pad 15: unconnected-(J2-Pin_15-Pad15) -> /CS14
- J2 pad 16: unconnected-(J2-Pin_16-Pad16) -> /CS15
- J2 pad 17: unconnected-(J2-Pin_17-Pad17) -> /CS16
- J2 pad 18: unconnected-(J2-Pin_18-Pad18) -> /CS17
- J2 pad 19: unconnected-(J2-Pin_19-Pad19) -> /CS18
- J2 pad 2: unconnected-(J2-Pin_2-Pad2) -> /CS1
- J2 pad 20: unconnected-(J2-Pin_20-Pad20) -> /CS19
- J2 pad 3: unconnected-(J2-Pin_3-Pad3) -> /CS2
- J2 pad 4: unconnected-(J2-Pin_4-Pad4) -> /CS3
- J2 pad 5: unconnected-(J2-Pin_5-Pad5) -> /CS4
- J2 pad 6: unconnected-(J2-Pin_6-Pad6) -> /CS5
- J2 pad 7: unconnected-(J2-Pin_7-Pad7) -> /CS6
- J2 pad 8: unconnected-(J2-Pin_8-Pad8) -> /CS7
- J2 pad 9: unconnected-(J2-Pin_9-Pad9) -> /CS8
- J3 pad 1: unconnected-(J3-Pin_1-Pad1) -> +5V
Other:
- board size 95 x 66 mm -> 95 x 70 mm
- copper layers 2 -> 4

Commit message: update
Parts:
- added U4: 74HC688, Package_SO:SOIC-20W_7.5x12.8mm_P1.27mm, F.Cu at (168.0, 80.3)
- moved U2 15.2 mm to (152.8, 80.2)
Connections:
- J4 pad 10: /PA7 -> /PA7A
- J4 pad 13: /PA0 -> /PB0A
- J4 pad 14: unconnected-(J4-Pin_14-Pad14) -> /PB1A
- J4 pad 15: /PA2 -> /PB2A
- J4 pad 16: unconnected-(J4-Pin_16-Pad16) -> /PB3A
- J4 pad 17: /PA4 -> /PB4A
- J4 pad 18: unconnected-(J4-Pin_18-Pad18) -> /PB5A
- J4 pad 19: /PA6 -> /PB6A
- J4 pad 20: unconnected-(J4-Pin_20-Pad20) -> /PB7A
- J4 pad 22: unconnected-(J4-Pin_22-Pad22) -> +5V
- J4 pad 23: /PA0 -> /PC0A
- J4 pad 24: unconnected-(J4-Pin_24-Pad24) -> /PC1A
- J4 pad 25: /PA2 -> /PC2A
- J4 pad 26: unconnected-(J4-Pin_26-Pad26) -> /PC3A
- J4 pad 27: /PA4 -> /PC4A
- J4 pad 28: unconnected-(J4-Pin_28-Pad28) -> /PC5A
- J4 pad 29: /PA6 -> /PC6A
- J4 pad 3: /PA0 -> /PA0A
- J4 pad 30: unconnected-(J4-Pin_30-Pad30) -> /PC7A
- J4 pad 4: /PA1 -> /PA1A
- J4 pad 5: /PA2 -> /PA2A
- J4 pad 6: /PA3 -> /PA3A
- J4 pad 7: /PA4 -> /PA4A
- J4 pad 8: /PA5 -> /PA5A
- J4 pad 9: /PA6 -> /PA6A
- J5 pad 10: /PA7 -> /PA7B
- J5 pad 13: /PA0 -> /PB0B
- J5 pad 14: unconnected-(J5-Pin_14-Pad14) -> /PB1B
- J5 pad 15: /PA2 -> /PB2B
- J5 pad 16: unconnected-(J5-Pin_16-Pad16) -> /PB3B
- J5 pad 17: /PA4 -> /PB4B
- J5 pad 18: unconnected-(J5-Pin_18-Pad18) -> /PB5B
- J5 pad 19: /PA6 -> /PB6B
- J5 pad 20: unconnected-(J5-Pin_20-Pad20) -> /PB7B
- J5 pad 22: unconnected-(J5-Pin_22-Pad22) -> +5V
- J5 pad 23: /PA0 -> /PC0B
- J5 pad 24: unconnected-(J5-Pin_24-Pad24) -> /PC1B
- J5 pad 25: /PA2 -> /PC2B
- J5 pad 26: unconnected-(J5-Pin_26-Pad26) -> /PC3B
- J5 pad 27: /PA4 -> /PC4B
- J5 pad 28: unconnected-(J5-Pin_28-Pad28) -> /PC5B
- J5 pad 29: /PA6 -> /PC6B
- J5 pad 3: /PA0 -> /PA0B
- J5 pad 30: unconnected-(J5-Pin_30-Pad30) -> /PC7B
- J5 pad 4: /PA1 -> /PA1B
- J5 pad 5: /PA2 -> /PA2B
- J5 pad 6: /PA3 -> /PA3B
- J5 pad 7: /PA4 -> /PA4B
- J5 pad 8: /PA5 -> /PA5B
- J5 pad 9: /PA6 -> /PA6B
- U1 pad 10: /PC7 -> /PC7A
- U1 pad 11: /PC6 -> /PC6A
- U1 pad 12: /PC5 -> /PC5A
- U1 pad 13: /PC4 -> /PC4A
- U1 pad 14: /PC0 -> /PC0A
- U1 pad 15: /PC1 -> /PC1A
- U1 pad 16: /PC2 -> /PC2A
- U1 pad 17: /PC3 -> /PC3A
- U1 pad 18: /PB0 -> /PB0A
- U1 pad 19: /PB1 -> /PB1A
- U1 pad 20: /PB2 -> /PB2A
- U1 pad 21: /PB3 -> /PB3A
- U1 pad 22: /PB4 -> /PB4A
- U1 pad 23: /PB5 -> /PB5A
- U1 pad 24: /PB6 -> /PB6A
- U1 pad 25: /PB7 -> /PB7A
- U1 pad 35: unconnected-(U1-RESET-Pad35) -> /RESET
- U1 pad 37: /PA7 -> /PA7A
- U1 pad 38: /PA6 -> /PA6A
- U1 pad 39: /PA5 -> /PA5A
- U1 pad 40: /PA4 -> /PA4A
- U1 pad 6: Net-(U1-~{CS}) -> /CS0
- U2 pad 19: Net-(U1-~{CS}) -> /CS0
- U3 pad 1: /PA3 -> /PA3B
- U3 pad 10: /PC7 -> /PC7B
- U3 pad 11: /PC6 -> /PC6B
- U3 pad 12: /PC5 -> /PC5B
- U3 pad 13: /PC4 -> /PC4B
- U3 pad 14: /PC0 -> /PC0B
- U3 pad 15: /PC1 -> /PC1B
- U3 pad 16: /PC2 -> /PC2B
- U3 pad 17: /PC3 -> /PC3B
- U3 pad 18: /PB0 -> /PB0B
- U3 pad 19: /PB1 -> /PB1B
- U3 pad 2: /PA2 -> /PA2B
- U3 pad 20: /PB2 -> /PB2B
- U3 pad 21: /PB3 -> /PB3B
- U3 pad 22: /PB4 -> /PB4B
- U3 pad 23: /PB5 -> /PB5B
- U3 pad 24: /PB6 -> /PB6B
- U3 pad 25: /PB7 -> /PB7B
- U3 pad 3: /PA1 -> /PA1B
- U3 pad 35: unconnected-(U3-RESET-Pad35) -> /RESET
- U3 pad 37: /PA7 -> /PA7B
- U3 pad 38: /PA6 -> /PA6B
- U3 pad 39: /PA5 -> /PA5B
- U3 pad 4: /PA0 -> /PA0B
- U3 pad 40: /PA4 -> /PA4B
- U3 pad 6: unconnected-(U3-~{CS}-Pad6) -> /CS1
Routing:
- net /D0: track 0.00 -> 102.5 mm, vias 0 -> 1
- net /PB1A: track 0.00 -> 69.9 mm, vias 0 -> 2
- net /PB0A: track 0.00 -> 65.5 mm, vias 0 -> 2
- net /D1: track 0.00 -> 65.2 mm
- net /D2: track 0.00 -> 65.2 mm
- net /D3: track 0.00 -> 65.1 mm
- net /PA7A: track 0.00 -> 22.2 mm, vias 0 -> 1
- net /PA5A: track 0.00 -> 19.6 mm, vias 0 -> 1
- net /PB5A: track 0.00 -> 18.1 mm
- net /PA0A: track 0.00 -> 18.0 mm, vias 0 -> 1
- net /PB3A: track 0.00 -> 17.8 mm
- net /PA1A: track 0.00 -> 17.3 mm, vias 0 -> 1
- net /PA2A: track 0.00 -> 15.4 mm, vias 0 -> 1
- net /PA6A: track 0.00 -> 15.3 mm, vias 0 -> 1
- net /PB4A: track 0.00 -> 15.1 mm
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