File: 8052-IO.kicad_sch (KiCad schematic)
At the start: 7 parts, among them J1 Conn_01x20_Pin, J2 Conn_01x20_Pin, J3 Conn_02x25_Odd_Even

Commit message: update
Parts:
- added J4: Conn_02x15_Odd_Even, Connector_PinHeader_2.54mm:PinHeader_2x15_P2.54mm_Horizontal, symbol Connector_Generic:Conn_02x15_Odd_Even
- added J5: Conn_02x16_Odd_Even, Connector_PinHeader_2.54mm:PinHeader_2x15_P2.54mm_Horizontal, symbol Connector_Generic:Conn_02x15_Odd_Even
- added U1, U3: 82C55A, Package_DIP:DIP-40_W15.24mm, symbol Interface:82C55A
- added U2: 74HC688, Package_SO:SOIC-20W_7.5x12.8mm_P1.27mm, symbol 74xx:74HC688
Connections:
- net +5V: now also J3.1 (Pin_1), J4.12 (Pin_12), J4.2 (Pin_2), J5.12 (Pin_12), J5.2 (Pin_2), U1.26 (VCC), U2.20 (VCC), U3.26 (VCC)
- net A0: now also U1.9 (A0), U3.9 (A0)
- net A1: now also U1.8 (A1), U3.8 (A1)
- net A10: now also U2.15 (P6)
- net A11: now also U2.17 (P7)
- net A4: now also U2.2 (P0)
- net A5: now also U2.4 (P1)
- net A6: now also U2.6 (P2)
- net A7: now also U2.8 (P3)
- net A8: now also U2.11 (P4)
- net A9: now also U2.13 (P5)
- net D0: now also U1.34 (D0), U3.34 (D0)
- net D1: now also U1.33 (D1), U3.33 (D1)
- net D2: now also U1.32 (D2), U3.32 (D2)
- net D3: now also U1.31 (D3), U3.31 (D3)
- net D4: now also U1.30 (D4), U3.30 (D4)
- net D5: now also U1.29 (D5), U3.29 (D5)
- net D6: now also U1.28 (D6), U3.28 (D6)
- net D7: now also U1.27 (D7), U3.27 (D7)
- net GND: now also J4.1 (Pin_1), J4.11 (Pin_11), J4.21 (Pin_21), J5.1 (Pin_1), J5.11 (Pin_11), J5.21 (Pin_21), U1.7 (GND), U2.10 (GND), U3.7 (GND)
- net ~{RD}: now also U1.36 (~{WR}), U3.36 (~{WR}); no longer J1.17 (Pin_17)
- net ~{WR}: now also U1.5 (~{RD}), U3.5 (~{RD}); no longer J1.16 (Pin_16)
- net CS0: now reaches J2.1 (Pin_1)
- net CS9: now reaches J2.10 (Pin_10)
- net CS10: now reaches J2.11 (Pin_11)
- net CA11: now reaches J2.12 (Pin_12)
- net CS12: now reaches J2.13 (Pin_13)
- net CS13: now reaches J2.14 (Pin_14)
- net CS14: now reaches J2.15 (Pin_15)
- net CS15: now reaches J2.16 (Pin_16)
- net CS16: now reaches J2.17 (Pin_17)
- net CS17: now reaches J2.18 (Pin_18)
- net CS18: now reaches J2.19 (Pin_19)
- net CS1: now reaches J2.2 (Pin_2)
- net CS19: now reaches J2.20 (Pin_20)
- net CS2: now reaches J2.3 (Pin_3)
- net CS3: now reaches J2.4 (Pin_4)
- net CS4: now reaches J2.5 (Pin_5)
- net CS5: now reaches J2.6 (Pin_6)
- net CS6: now reaches J2.7 (Pin_7)
- net CS7: now reaches J2.8 (Pin_8)
- net CS8: now reaches J2.9 (Pin_9)
- new net: U1.6 (~{CS}), U2.19 (P=R)
- new net PA0: J4.13 (Pin_13), J4.23 (Pin_23), J4.3 (Pin_3), J5.13 (Pin_13), J5.23 (Pin_23), J5.3 (Pin_3), U3.4 (PA0)
- new net PA0A: U1.4 (PA0)
- new net PA1: J4.4 (Pin_4), J5.4 (Pin_4), U3.3 (PA1)
- new net PA1A: U1.3 (PA1)
- new net PA2: J4.15 (Pin_15), J4.25 (Pin_25), J4.5 (Pin_5), J5.15 (Pin_15), J5.25 (Pin_25), J5.5 (Pin_5), U3.2 (PA2)
- new net PA2A: U1.2 (PA2)
- new net PA3: J4.6 (Pin_6), J5.6 (Pin_6), U3.1 (PA3)
- new net PA3A: U1.1 (PA3)
- new net PA4: J4.17 (Pin_17), J4.27 (Pin_27), J4.7 (Pin_7), J5.17 (Pin_17), J5.27 (Pin_27), J5.7 (Pin_7), U1.40 (PA4), U3.40 (PA4)
- new net PA5: J4.8 (Pin_8), J5.8 (Pin_8), U1.39 (PA5), U3.39 (PA5)
- new net PA6: J4.19 (Pin_19), J4.29 (Pin_29), J4.9 (Pin_9), J5.19 (Pin_19), J5.29 (Pin_29), J5.9 (Pin_9), U1.38 (PA6), U3.38 (PA6)
- new net PA7: J4.10 (Pin_10), J5.10 (Pin_10), U1.37 (PA7), U3.37 (PA7)
- new net PB0: U1.18 (PB0), U3.18 (PB0)
- new net PB1: U1.19 (PB1), U3.19 (PB1)
- new net PB2: U1.20 (PB2), U3.20 (PB2)
- new net PB3: U1.21 (PB3), U3.21 (PB3)
- new net PB4: U1.22 (PB4), U3.22 (PB4)
- new net PB5: U1.23 (PB5), U3.23 (PB5)
- new net PB6: U1.24 (PB6), U3.24 (PB6)
- new net PB7: U1.25 (PB7), U3.25 (PB7)
- new net PC0: U1.14 (PC0), U3.14 (PC0)
- new net PC1: U1.15 (PC1), U3.15 (PC1)
- new net PC2: U1.16 (PC2), U3.16 (PC2)
- new net PC3: U1.17 (PC3), U3.17 (PC3)
- new net PC4: U1.13 (PC4), U3.13 (PC4)
- new net PC5: U1.12 (PC5), U3.12 (PC5)
- new net PC6: U1.11 (PC6), U3.11 (PC6)
- new net PC7: U1.10 (PC7), U3.10 (PC7)
Other:
- moved on the sheet: H1, H2, H3, H4, J1, J2, J3

Commit message: update
Parts:
- added U4: 74HC688, Package_SO:SOIC-20W_7.5x12.8mm_P1.27mm, symbol 74xx:74HC688
Connections:
- net +5V: now also J4.22 (Pin_22), J5.22 (Pin_22), U4.20 (VCC)
- net A10: now also U4.15 (P6)
- net A11: now also U4.17 (P7)
- net A4: now also U4.2 (P0)
- net A5: now also U4.4 (P1)
- net A6: now also U4.6 (P2)
- net A7: now also U4.8 (P3)
- net A8: now also U4.11 (P4)
- net A9: now also U4.13 (P5)
- net CS0: now also U1.6 (~{CS}), U2.19 (P=R)
- net CS1: now also U3.6 (~{CS}), U4.19 (P=R)
- net GND: now also U4.10 (GND)
- net PA0A: now also J4.3 (Pin_3)
- net PA1A: now also J4.4 (Pin_4)
- net PA2A: now also J4.5 (Pin_5)
- net PA3A: now also J4.6 (Pin_6)
- net RESET: now also U1.35 (RESET), U3.35 (RESET)
- net PB1B: now reaches J5.14 (Pin_14)
- net PB1B: now also U3.19 (PB1)
- net PB3B: now reaches J5.16 (Pin_16)
- net PB3B: now also U3.21 (PB3)
- net PB5B: now reaches J5.18 (Pin_18)
- net PB5B: now also U3.23 (PB5)
- net PB7B: now reaches J5.20 (Pin_20)
- net PB7B: now also U3.25 (PB7)
- net PC1B: now reaches J5.24 (Pin_24)
- net PC1B: now also U3.15 (PC1)
- net PC3B: now reaches J5.26 (Pin_26)
- net PC3B: now also U3.17 (PC3)
- net PC5B: now reaches J5.28 (Pin_28)
- net PC5B: now also U3.12 (PC5)
- net PC7B: now reaches J5.30 (Pin_30)
- net PC7B: now also U3.10 (PC7)
- net PB1A: now reaches J4.14 (Pin_14)
- net PB1A: now also U1.19 (PB1)
- net PB3A: now reaches J4.16 (Pin_16)
- net PB3A: now also U1.21 (PB3)
- net PB5A: now reaches J4.18 (Pin_18)
- net PB5A: now also U1.23 (PB5)
- net PB7A: now reaches J4.20 (Pin_20)
- net PB7A: now also U1.25 (PB7)
- net PC1A: now reaches J4.24 (Pin_24)
- net PC1A: now also U1.15 (PC1)
- net PC3A: now reaches J4.26 (Pin_26)
- net PC3A: now also U1.17 (PC3)
- net PC5A: now reaches J4.28 (Pin_28)
- net PC5A: now also U1.12 (PC5)
- net PC7A: now reaches J4.30 (Pin_30)
- net PC7A: now also U1.10 (PC7)
- removed net PA0: J4.13 (Pin_13), J4.23 (Pin_23), J4.3 (Pin_3), J5.13 (Pin_13), J5.23 (Pin_23), J5.3 (Pin_3), U3.4 (PA0)
- net PA1 renamed PA1B
- net PA1B: no longer J4.4 (Pin_4)
- removed net PA2: J4.15 (Pin_15), J4.25 (Pin_25), J4.5 (Pin_5), J5.15 (Pin_15), J5.25 (Pin_25), J5.5 (Pin_5), U3.2 (PA2)
- net PA3 renamed PA3B
- net PA3B: no longer J4.6 (Pin_6)
- removed net PA4: J4.17 (Pin_17), J4.27 (Pin_27), J4.7 (Pin_7), J5.17 (Pin_17), J5.27 (Pin_27), J5.7 (Pin_7), U1.40 (PA4), U3.40 (PA4)
- net PA5 renamed PA5A
- net PA5A: no longer J5.8 (Pin_8), U3.39 (PA5)
- removed net PA6: J4.19 (Pin_19), J4.29 (Pin_29), J4.9 (Pin_9), J5.19 (Pin_19), J5.29 (Pin_29), J5.9 (Pin_9), U1.38 (PA6), U3.38 (PA6)
- net PA7 renamed PA7A
- net PA7A: no longer J5.10 (Pin_10), U3.37 (PA7)
- net PB0 renamed PB0A
- net PB0A: now also J4.13 (Pin_13); no longer U3.18 (PB0)
- removed net PB1: U1.19 (PB1), U3.19 (PB1)
- net PB2 renamed PB2A
- net PB2A: now also J4.15 (Pin_15); no longer U3.20 (PB2)
- removed net PB3: U1.21 (PB3), U3.21 (PB3)
- net PB4 renamed PB4A
- net PB4A: now also J4.17 (Pin_17); no longer U3.22 (PB4)
- removed net PB5: U1.23 (PB5), U3.23 (PB5)
- net PB6 renamed PB6A
- net PB6A: now also J4.19 (Pin_19); no longer U3.24 (PB6)
- removed net PB7: U1.25 (PB7), U3.25 (PB7)
- net PC0 renamed PC0A
- net PC0A: now also J4.23 (Pin_23); no longer U3.14 (PC0)
- removed net PC1: U1.15 (PC1), U3.15 (PC1)
- net PC2 renamed PC2A
- net PC2A: now also J4.25 (Pin_25); no longer U3.16 (PC2)
- removed net PC3: U1.17 (PC3), U3.17 (PC3)
- net PC4 renamed PC4A
- net PC4A: now also J4.27 (Pin_27); no longer U3.13 (PC4)
- removed net PC5: U1.12 (PC5), U3.12 (PC5)
- net PC6 renamed PC6A
- net PC6A: now also J4.29 (Pin_29); no longer U3.11 (PC6)
- removed net PC7: U1.10 (PC7), U3.10 (PC7)
- new net PA0B: J5.3 (Pin_3), U3.4 (PA0)
- new net PA2B: J5.5 (Pin_5), U3.2 (PA2)
- new net PA4A: J4.7 (Pin_7), U1.40 (PA4)
- new net PA4B: J5.7 (Pin_7), U3.40 (PA4)
- new net PA5B: J5.8 (Pin_8), U3.39 (PA5)
- new net PA6A: J4.9 (Pin_9), U1.38 (PA6)
- new net PA6B: J5.9 (Pin_9), U3.38 (PA6)
- new net PA7B: J5.10 (Pin_10), U3.37 (PA7)
- new net PB0B: J5.13 (Pin_13), U3.18 (PB0)
- new net PB2B: J5.15 (Pin_15), U3.20 (PB2)
- new net PB4B: J5.17 (Pin_17), U3.22 (PB4)
- new net PB6B: J5.19 (Pin_19), U3.24 (PB6)
- new net PC0B: J5.23 (Pin_23), U3.14 (PC0)
- new net PC2B: J5.25 (Pin_25), U3.16 (PC2)
- new net PC4B: J5.27 (Pin_27), U3.13 (PC4)
- new net PC6B: J5.29 (Pin_29), U3.11 (PC6)
